File: GPS_Module.kicad_sch (KiCad schematic)
At the start: 0 parts

Commit message: test
Parts:
- added U6: SAM-M8Q, RF_GPS:ublox_SAM-M8Q, symbol RF_GPS:SAM-M8Q
Connections:
- new net: U6.1 (GND), U6.10 (GND), U6.11 (GND), U6.15 (GND), U6.16 (GND), U6.20 (GND), U6.4 (GND), U6.5 (GND), U6.6 (GND)
Changed lines of the file:
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@@
 	(generator_version "9.0")
 	(paper "A4")
+	(symbol
+		(lib_id "RF_GPS:SAM-M8Q")
+		(at 104.14 71.12 0)
+		(unit 1)
+		(exclude_from_sim no)
+		(in_bom yes)
+		(on_board yes)
+		(dnp no)
+		(fields_autoplaced yes)
+		(property "Reference" "U6"
+			(at 106.2833 83.82 0)
+			(effects
+				(font
+					(size 1.27 1.27)
+				)
+				(justify left)
+			)
+		)
+		(property "Value" "SAM-M8Q"
+			(at 106.2833 86.36 0)
+			(effects
+				(font
+					(size 1.27 1.27)
+				)
+				(justify left)
+			)
+		)
+		(property "Footprint" "RF_GPS:ublox_SAM-M8Q"
+			(at 116.84 82.55 0)
+			(effects
+				(font
+					(size 1.27 1.27)
+				)
+				(hide yes)
+			)
+		)
+		(property "Datasheet" "https://www.u-blox.com/sites/default/files/SAM-M8Q_DataSheet_%28UBX-16012619%29.pdf"
+			(at 104.14 71.12 0)
+			(effects
+				(font
+					(size 1.27 1.27)
+				)
+				(hide yes)
+			)
+		)
+		(property "Description" "GPS ublox M8 variant"
+			(at 104.14 71.12 0)
+			(effects
+				(font
+					(size 1.27 1.27)
+				)
+				(hide yes)
+			)
+		)
+		(pin "17"
+		)
+		(pin "7"
+		)
+		(pin "13"
+		)
+		(pin "8"
+		)
+		(pin "19"
+		)
+		(pin "18"
+		)
+		(pin "10"
+		)
+		(pin "11"
+		)
+		(pin "20"
+		)
+		(pin "4"
+		)
+		(pin "5"
+		)
+		(pin "6"
+		)
+		(pin "3"
+		)
+		(pin "14"
+		)
+		(pin "1"
+		)
+		(pin "2"
+		)
+		(pin "16"
+		)
+		(pin "15"
+		)
+		(pin "12"
+		)
+		(pin "9"
+		)
+		(instances
+			(project ""
+				(path "/5b969f6e-a36e-432b-8f00-b2d6a515a877/86749ea3-b799-4cf0-94d1-46de6ccb32b0"
+					(reference "U6")
+					(unit 1)
+				)
+			)
+		)
+	)
 )
