File: Power.kicad_sch (KiCad schematic)
At the start: 0 parts

Commit message: test
Parts:
- added D1: B_LED, LED_SMD:LED_0603_1608Metric, symbol Device:LED
- added R10: 220, Resistor_SMD:R_0603_1608Metric, symbol Device:R
- added U5: BQ25798RQMR, RQM0029A-MFG, symbol BQ25798RQMR:BQ25798RQMR
Connections:
- new net: D1.2 (A), R10.2
- new net GND: D1.1 (K), U5.10 (ACDRV2), U5.11 (ACDRV1)
