File: hardware/GOG.kicad_sch (KiCad schematic)
At the start: 0 parts

Commit message: Found all diodes & transistors footprint & JLCPCB
Other:
- company: (none) -> ECAM Brussels Engineering School
Changed lines of the file:
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@@
 	(generator_version "9.0")
 	(paper "A4")
+	(title_block
+		(rev "0.1")
+		(company "ECAM Brussels Engineering School")
+	)
 	(sheet
 		(at 34.29 39.37)
