File: hardware/GOG.kicad_pcb (KiCad board)
At the start: 2 copper layers, 0 parts

Commit message: First draft
Parts:
- added C1: 10µF, Capacitor_SMD:C_0603_1608Metric, F.Cu at (133.3, 55.2)
- added C10: 0.1u, Capacitor_SMD:C_0402_1005Metric, F.Cu at (156.2, 106.0)
- added C11: 0.1u, Capacitor_SMD:C_0402_1005Metric, F.Cu at (131.7, 111.9)
- added C12: 0.1u, Capacitor_SMD:C_0603_1608Metric, F.Cu at (171.9, 71.8)
- added C13: 0.1u, Capacitor_SMD:C_0603_1608Metric, F.Cu at (153.5, 71.2)
- added C14: 22u, Capacitor_SMD:C_0805_2012Metric, F.Cu at (167.9, 73.3)
- added C15: 22u, Capacitor_SMD:C_0805_2012Metric, F.Cu at (149.4, 73.0)
- added C16: 22u, Capacitor_SMD:C_0805_2012Metric, F.Cu at (167.9, 71.3)
- added C17: 22u, Capacitor_SMD:C_0805_2012Metric, F.Cu at (149.4, 71.0)
- added C18: 10u, Capacitor_SMD:C_0805_2012Metric, F.Cu at (152.2, 100.0)
- added C19: 10u, Capacitor_SMD:C_0805_2012Metric, F.Cu at (152.2, 102.0)
- added C2: 0.1µF, Capacitor_SMD:C_0603_1608Metric, F.Cu at (133.2, 53.5)
- added C20: 0.1u, Capacitor_SMD:C_0402_1005Metric, F.Cu at (152.0, 103.5)
- added C21: 0.1u, Capacitor_SMD:C_0402_1005Metric, F.Cu at (155.7, 96.8)
- added C22: 0.1u, Capacitor_SMD:C_0402_1005Metric, F.Cu at (159.4, 97.0)
- added C23: 10u, Capacitor_SMD:C_0805_2012Metric, F.Cu at (155.7, 95.3)
- added C24: 10u, Capacitor_SMD:C_0805_2012Metric, F.Cu at (159.4, 95.3)
- added C25: 4.7u, Capacitor_SMD:C_0603_1608Metric, F.Cu at (152.7, 106.5)
- added C26: 10u, Capacitor_SMD:C_0805_2012Metric, F.Cu at (155.7, 93.3)
- added C27: 10u, Capacitor_SMD:C_0805_2012Metric, F.Cu at (159.4, 93.3)
- added C28: 47n, Capacitor_SMD:C_0603_1608Metric, F.Cu at (152.7, 105.0)
- added C29: 47n, Capacitor_SMD:C_0603_1608Metric, F.Cu at (163.2, 98.5)
- added C3: 1µF, Capacitor_SMD:C_0603_1608Metric, F.Cu at (132.5, 58.8)
- added C30: 10u, Capacitor_SMD:C_0805_2012Metric, F.Cu at (155.7, 91.3)
- added C31: 10u, Capacitor_SMD:C_0805_2012Metric, F.Cu at (159.4, 91.3)
- added C32: 1n, Capacitor_SMD:C_0402_1005Metric, F.Cu at (162.7, 100.8)
- added C33: 10u, Capacitor_SMD:C_0805_2012Metric, F.Cu at (159.4, 89.3)
- added C34: 10u, Capacitor_SMD:C_0805_2012Metric, F.Cu at (159.4, 87.3)
- added C35: 10u, Capacitor_SMD:C_0805_2012Metric, F.Cu at (164.8, 105.1)
- added C36: 10u, Capacitor_SMD:C_0805_2012Metric, F.Cu at (164.8, 103.0)
- added C4: 100nF, Capacitor_SMD:C_0201_0603Metric, F.Cu at (135.5, 132.2)
- added C5: C, Capacitor_SMD:C_0805_2012Metric_Pad1.18x1.45mm_HandSolder, F.Cu at (123.5, 143.8)
- added C6: C, Capacitor_SMD:C_0805_2012Metric_Pad1.18x1.45mm_HandSolder, F.Cu at (125.5, 147.5)
- added C7: 1µF, Capacitor_SMD:C_0603_1608Metric, F.Cu at (180.5, 118.3)
- added C8: 10u, Capacitor_SMD:C_0805_2012Metric, F.Cu at (167.9, 75.3)
- added C9: 10u, Capacitor_SMD:C_0805_2012Metric, F.Cu at (149.4, 75.0)
- added D1: R_LED, LED_SMD:LED_0603_1608Metric, F.Cu at (127.0, 51.8)
- added D2: R_LED, LED_SMD:LED_0603_1608Metric, F.Cu at (176.8, 143.3)
- added D3: D_Zener, Diode_SMD:D_SOD-123, F.Cu at (131.7, 109.9)
- added D4: D_Zener, Diode_SMD:D_SOD-123, F.Cu at (141.4, 106.6)
- added D5: D_Zener, Diode_SMD:D_SOD-123, F.Cu at (146.4, 114.7)
- added D6: LED, LED_SMD:LED_0603_1608Metric, F.Cu at (148.5, 95.8)
- added J1: USB_C_Receptacle_USB2.0_16P, Connector_USB:USB_C_Receptacle_GCT_USB4105-xx-A_16P_TopMnt_Horizontal, F.Cu at (196.2, 62.2)
- added J10: Conn_01x02, Connector_PinHeader_2.54mm:PinHeader_1x02_P2.54mm_Vertical, F.Cu at (157.0, 117.0)
- added J11: Conn_01x02, Connector_JST:JST_XH_B2B-XH-A_1x02_P2.50mm_Vertical, F.Cu at (185.5, 94.0)
- added J2: Conn_01x02_Pin, Connector_PinHeader_2.54mm:PinHeader_1x02_P2.54mm_Vertical, F.Cu at (176.5, 53.2)
- added J3: Conn_01x04_Pin, Connector_PinHeader_2.54mm:PinHeader_1x04_P2.54mm_Vertical, F.Cu at (129.1, 66.0)
- added J4: Conn_01x02_Pin, Connector_PinHeader_2.54mm:PinHeader_1x02_P2.54mm_Vertical, F.Cu at (185.5, 53.2)
- added J5: 85201239, SMA-85201239:HUBER_SUHNER_85201239, F.Cu at (147.8, 143.7)
- added J6: Conn_01x04_Pin, Connector_JST:JST_XA_B04B-XASK-1_1x04_P2.50mm_Vertical, F.Cu at (193.5, 110.8)
- added J7: Conn_01x04_Pin, Connector_JST:JST_XA_B04B-XASK-1_1x04_P2.50mm_Vertical, F.Cu at (193.5, 145.6)
- added J8: Screw_Terminal_01x02, GoG_Library:TerminalBlock_WJ126V-5.0-2P_1x02_P5.00mm, F.Cu at (106.5, 102.8)
- added J9: Conn_01x04, Connector_PinHeader_2.54mm:PinHeader_1x04_P2.54mm_Vertical, F.Cu at (159.7, 80.2)
- added L1: 3.9u, Inductor_SMD:L_Sunlord_SWPA4030S, F.Cu at (176.6, 74.0)
- added L2: 4.7u, Inductor_SMD:L_Sunlord_SWPA4030S, F.Cu at (158.5, 73.8)
- added L3: 2.2u, GoG_Library:MDA5030-2R2M, F.Cu at (140.8, 95.7)
- added Q1: Q_PMOS, Package_TO_SOT_SMD:SOT-23, F.Cu at (131.7, 105.1)
- added Q2: Q_NMOS, Package_TO_SOT_SMD:SOT-23, F.Cu at (144.7, 106.6)
- added Q3: Q_NMOS, Package_TO_SOT_SMD:SOT-23, F.Cu at (138.4, 106.7)
- added Q4: Q_NMOS, Package_TO_SOT_SMD:SOT-23, F.Cu at (149.4, 115.0)
- added Q5: Q_NMOS, Package_TO_SOT_SMD:SOT-23, F.Cu at (143.2, 114.9)
- added R1: 5k1, Resistor_SMD:R_0603_1608Metric, F.Cu at (168.2, 61.8)
- added R10: 1k, Resistor_SMD:R_0603_1608Metric, F.Cu at (176.8, 139.3)
- added R11: 470, Resistor_SMD:R_0603_1608Metric, F.Cu at (194.0, 126.8)
- added R12: 470, Resistor_SMD:R_0603_1608Metric, F.Cu at (193.9, 128.6)
- added R13: 22, Resistor_SMD:R_0603_1608Metric, F.Cu at (180.5, 142.6)
- added R14: 22, Resistor_SMD:R_0603_1608Metric, F.Cu at (193.9, 130.6)
- added R15: 0, Resistor_SMD:R_1206_3216Metric, F.Cu at (127.0, 105.6)
- added R16: 100k, Resistor_SMD:R_0402_1005Metric, F.Cu at (127.9, 109.9)
- added R17: 5.1k, Resistor_SMD:R_0402_1005Metric, F.Cu at (155.8, 113.8)
- added R18: 30k, Resistor_SMD:R_0402_1005Metric, F.Cu at (162.5, 112.5)
- added R19: 120k, Resistor_SMD:R_0402_1005Metric, F.Cu at (155.8, 112.8)
- added R2: 5k1, Resistor_SMD:R_0603_1608Metric, F.Cu at (170.8, 61.8)
- added R20: 100k, Resistor_SMD:R_0402_1005Metric, F.Cu at (162.5, 111.5)
- added R21: 2.2k, Resistor_SMD:R_0402_1005Metric, F.Cu at (145.9, 95.8)
- added R22: 300, Resistor_SMD:R_0603_1608Metric, F.Cu at (141.4, 102.6)
- added R23: 300, Resistor_SMD:R_0603_1608Metric, F.Cu at (146.4, 118.6)
- added R24: 10k, Resistor_SMD:R_0402_1005Metric, F.Cu at (160.5, 106.0)
- added R25: 8.2k, Resistor_SMD:R_0402_1005Metric, F.Cu at (162.7, 99.8)
- added R26: 100, Resistor_SMD:R_0402_1005Metric, F.Cu at (164.0, 106.5)
- added R3: 1k, Resistor_SMD:R_0603_1608Metric, F.Cu at (133.3, 51.8)
- added R4: 10k, Resistor_SMD:R_0603_1608Metric, F.Cu at (164.0, 55.8)
- added R5: 10k, Resistor_SMD:R_0603_1608Metric, F.Cu at (136.5, 58.8)
- added R6: 10k, Resistor_SMD:R_0603_1608Metric, F.Cu at (134.5, 58.8)
- added R7: 4.7k, Resistor_SMD:R_0603_1608Metric, F.Cu at (168.8, 55.8)
- added R8: 4.7k, Resistor_SMD:R_0603_1608Metric, F.Cu at (166.8, 55.8)
- added R9: 0, Resistor_SMD:R_0805_2012Metric_Pad1.20x1.40mm_HandSolder, F.Cu at (125.5, 143.8)
- added SW1: SW_Omron_B3FS, Button_Switch_SMD:SW_SPST_Omron_B3FS-100xP, F.Cu at (109.2, 55.2)
- added SW2: SW_Omron_B3FS, Button_Switch_SMD:SW_SPST_Omron_B3FS-100xP, F.Cu at (109.2, 65.0)
- added TH1: 10k, GoG_Library:Thermistor NTC, F.Cu at (162.6, 116.0)
- added TP1: TestPoint_2Pole, Connector_PinHeader_2.54mm:PinHeader_2x01_P2.54mm_Vertical, F.Cu at (115.7, 102.8)
- added TP10: TestPoint, TestPoint:TestPoint_Pad_D1.5mm, F.Cu at (142.2, 123.5)
- added TP11: TestPoint, TestPoint:TestPoint_Pad_D1.5mm, F.Cu at (156.8, 123.0)
- added TP12: TestPoint, TestPoint:TestPoint_Pad_D1.5mm, F.Cu at (144.5, 85.8)
- added TP13: TestPoint, TestPoint:TestPoint_Pad_D1.5mm, F.Cu at (162.5, 122.8)
- added TP14: TestPoint, TestPoint:TestPoint_Pad_D1.5mm, F.Cu at (172.2, 113.5)
- added TP15: TestPoint, TestPoint:TestPoint_Pad_D1.5mm, F.Cu at (131.8, 100.0)
- added TP16: TestPoint, TestPoint:TestPoint_Pad_D1.5mm, F.Cu at (131.8, 91.2)
- added TP17: TestPoint, TestPoint:TestPoint_Pad_D1.5mm, F.Cu at (150.8, 123.2)
- added TP18: TestPoint, TestPoint:TestPoint_Pad_D1.5mm, F.Cu at (160.5, 110.0)
- added TP19: TestPoint, TestPoint:TestPoint_Pad_D1.5mm, F.Cu at (148.5, 85.8)
- added TP2: TestPoint, TestPoint:TestPoint_Pad_D1.5mm, F.Cu at (121.5, 113.8)
- added TP20: TestPoint, TestPoint:TestPoint_Pad_D1.5mm, F.Cu at (152.2, 85.8)
- added TP21: TestPoint, TestPoint:TestPoint_Pad_D1.5mm, F.Cu at (155.8, 110.0)
- added TP22: TestPoint, TestPoint:TestPoint_Pad_D1.5mm, F.Cu at (172.2, 90.8)
- added TP23: TestPoint, TestPoint:TestPoint_Pad_D1.5mm, F.Cu at (172.2, 102.0)
- added TP24: TestPoint, TestPoint:TestPoint_Pad_D1.5mm, F.Cu at (172.2, 106.0)
- added TP25: TestPoint, TestPoint:TestPoint_Pad_D1.5mm, F.Cu at (172.2, 98.2)
- added TP26: TestPoint, TestPoint:TestPoint_Pad_D1.5mm, F.Cu at (172.2, 109.8)
- added TP27: TestPoint, TestPoint:TestPoint_Pad_D1.5mm, F.Cu at (131.8, 87.2)
- added TP28: TestPoint, TestPoint:TestPoint_Pad_D1.5mm, F.Cu at (172.2, 94.5)
- added TP29: TestPoint, TestPoint:TestPoint_Pad_D1.5mm, F.Cu at (150.2, 80.2)
- added TP3: TestPoint, TestPoint:TestPoint_Pad_D1.5mm, F.Cu at (176.4, 69.8)
- added TP4: TestPoint, TestPoint:TestPoint_Pad_D1.5mm, F.Cu at (158.5, 69.2)
- added TP5: TestPoint, TestPoint:TestPoint_Pad_D1.5mm, F.Cu at (121.5, 118.2)
- added TP6: TestPoint, TestPoint:TestPoint_Pad_D1.5mm, F.Cu at (186.8, 69.8)
- added TP7: TestPoint, TestPoint:TestPoint_Pad_D1.5mm, F.Cu at (131.8, 95.8)
- added TP8: TestPoint, TestPoint:TestPoint_Pad_D1.5mm, F.Cu at (135.2, 115.0)
- added TP9: TestPoint, TestPoint:TestPoint_Pad_D1.5mm, F.Cu at (135.2, 119.0)
- added TP_DIO1: TestPoint, TestPoint:TestPoint_Pad_D2.0mm, F.Cu at (147.5, 130.5)
- added TP_RESET1: TestPoint, TestPoint:TestPoint_Pad_D2.0mm, F.Cu at (110.8, 136.2)
- added TP_VCC_Lora1: TestPoint, TestPoint:TestPoint_Pad_D2.0mm, F.Cu at (147.5, 134.8)
- added U1: USBLC6-2SC6, Package_TO_SOT_SMD:SOT-23-6, F.Cu at (176.6, 61.9)
- added U2: ESP32-C3-WROOM-02, RF_Module:ESP32-C3-WROOM-02, F.Cu at (150.0, 57.0)
- added U3: RFM95W-868S2, RF_Module:HOPERF_RFM9XW_SMD, F.Cu at (124.2, 133.2)
- added U4: SAM-M8Q, RF_GPS:ublox_SAM-M8Q, F.Cu at (178.8, 128.8)
- added U5: AP63203WU, Package_TO_SOT_SMD:TSOT-23-6, F.Cu at (171.9, 74.5)
- added U6: AP63205WU, Package_TO_SOT_SMD:TSOT-23-6, F.Cu at (153.5, 74.2)
- added U7: BQ25798RQMR, BQ25798RQMR:RQM0029A-MFG, F.Cu at (158.1, 101.6)
Other:
- board outline added: 100 x 100 mm
