File: hardware/GOG.kicad_pcb (KiCad board)
At the start: 2 copper layers, 0 parts

Commit message: Fix several DRC errors & add all 3D models
Parts:
- added C1: 10µF, Capacitor_SMD:C_0603_1608Metric, F.Cu at (184.3, 85.5)
- added C10: 10u, Capacitor_SMD:C_0805_2012Metric, F.Cu at (249.3, 115.9)
- added C11: 10u, Capacitor_SMD:C_0805_2012Metric, F.Cu at (249.3, 118.9)
- added C12: 10u, Capacitor_SMD:C_0805_2012Metric, F.Cu at (249.3, 121.9)
- added C13: 10u, Capacitor_SMD:C_0805_2012Metric, F.Cu at (249.3, 124.9)
- added C14: 10u, Capacitor_SMD:C_0805_2012Metric, F.Cu at (249.3, 128.0)
- added C15: 0.1u, Capacitor_SMD:C_0402_1005Metric, F.Cu at (234.3, 150.2)
- added C16: 47n, Capacitor_SMD:C_0603_1608Metric, F.Cu at (262.4, 115.7)
- added C17: 4.7u, Capacitor_SMD:C_0603_1608Metric, F.Cu at (262.4, 118.2)
- added C18: 0.1u, Capacitor_SMD:C_0402_1005Metric, F.Cu at (234.3, 152.1)
- added C19: 47n, Capacitor_SMD:C_0603_1608Metric, F.Cu at (262.4, 120.7)
- added C2: 0.1µF, Capacitor_SMD:C_0603_1608Metric, F.Cu at (181.8, 85.5)
- added C20: 0.1u, Capacitor_SMD:C_0402_1005Metric, F.Cu at (234.3, 154.1)
- added C21: 10u, Capacitor_SMD:C_0805_2012Metric, F.Cu at (249.3, 131.0)
- added C22: 10u, Capacitor_SMD:C_0805_2012Metric, F.Cu at (249.3, 134.0)
- added C23: 10u, Capacitor_SMD:C_0805_2012Metric, F.Cu at (253.8, 115.9)
- added C24: 10u, Capacitor_SMD:C_0805_2012Metric, F.Cu at (253.8, 118.9)
- added C25: 10u, Capacitor_SMD:C_0805_2012Metric, F.Cu at (253.8, 121.9)
- added C26: 10u, Capacitor_SMD:C_0805_2012Metric, F.Cu at (253.8, 124.9)
- added C27: 10u, Capacitor_SMD:C_0805_2012Metric, F.Cu at (253.8, 128.0)
- added C28: 1n, Capacitor_SMD:C_0402_1005Metric, F.Cu at (234.3, 156.1)
- added C29: 0.1u, Capacitor_SMD:C_0603_1608Metric, F.Cu at (173.0, 152.2)
- added C3: 1µF, Capacitor_SMD:C_0603_1608Metric, F.Cu at (184.3, 88.0)
- added C30: 10u, Capacitor_SMD:C_0805_2012Metric, F.Cu at (168.3, 153.2)
- added C31: 22u, Capacitor_SMD:C_0805_2012Metric, F.Cu at (168.3, 156.2)
- added C32: 22u, Capacitor_SMD:C_0805_2012Metric, F.Cu at (173.3, 156.2)
- added C33: 0.1u, Capacitor_SMD:C_0603_1608Metric, F.Cu at (201.5, 160.9)
- added C34: 10u, Capacitor_SMD:C_0805_2012Metric, F.Cu at (197.2, 154.2)
- added C35: 22u, Capacitor_SMD:C_0805_2012Metric, F.Cu at (197.2, 157.2)
- added C36: 22u, Capacitor_SMD:C_0805_2012Metric, F.Cu at (197.2, 160.2)
- added C4: 100nF, Capacitor_SMD:C_0603_1608Metric, F.Cu at (119.5, 100.0)
- added C5: C, Resistor_SMD:R_0805_2012Metric_Pad1.20x1.40mm_HandSolder, F.Cu at (118.0, 96.0)
- added C6: C, Resistor_SMD:R_0805_2012Metric_Pad1.20x1.40mm_HandSolder, F.Cu at (111.0, 98.5)
- added C7: 1µF, Capacitor_SMD:C_0603_1608Metric, F.Cu at (118.0, 139.0)
- added C8: 0.1u, Capacitor_SMD:C_0402_1005Metric, F.Cu at (234.3, 146.2)
- added C9: 0.1u, Capacitor_SMD:C_0402_1005Metric, F.Cu at (234.3, 148.2)
- added D1: R_LED, LED_SMD:LED_0603_1608Metric, F.Cu at (190.3, 101.8)
- added D2: R_LED, LED_SMD:LED_0603_1608Metric, F.Cu at (131.8, 134.0)
- added D3: D_Zener, Diode_SMD:D_SOD-123, F.Cu at (267.4, 116.1)
- added D4: D_Zener, Diode_SMD:D_SOD-123, F.Cu at (267.4, 119.4)
- added D5: D_Zener, Diode_SMD:D_SOD-123, F.Cu at (267.4, 122.8)
- added D6: LED, LED_SMD:LED_0603_1608Metric, F.Cu at (242.9, 157.0)
- added J1: USB_C_Receptacle_USB2.0_16P, Connector_USB:USB_C_Receptacle_GCT_USB4105-xx-A_16P_TopMnt_Horizontal, F.Cu at (213.5, 112.4)
- added J10: Conn_01x04, Connector_PinHeader_2.54mm:PinHeader_1x04_P2.54mm_Vertical, F.Cu at (290.1, 133.6)
- added J11: Conn_01x02, Connector_PinHeader_2.54mm:PinHeader_1x02_P2.54mm_Vertical, F.Cu at (283.1, 134.1)
- added J2: Conn_01x02_Pin, Connector_PinHeader_2.54mm:PinHeader_1x02_P2.54mm_Vertical, F.Cu at (212.5, 96.3)
- added J3: Conn_01x04_Pin, Connector_PinHeader_2.54mm:PinHeader_1x04_P2.54mm_Vertical, F.Cu at (173.8, 86.0)
- added J4: Conn_01x02_Pin, Connector_PinHeader_2.54mm:PinHeader_1x02_P2.54mm_Vertical, F.Cu at (212.5, 103.3)
- added J5: 85201239, SMA-85201239:HUBER_SUHNER_85201239, F.Cu at (104.0, 97.5)
- added J6: Conn_01x04_Pin, Connector_JST:JST_XH_B4B-XH-A_1x04_P2.50mm_Vertical, F.Cu at (103.0, 119.0)
- added J7: Conn_01x04_Pin, Connector_JST:JST_XH_B4B-XH-A_1x04_P2.50mm_Vertical, F.Cu at (116.5, 143.5)
- added J8: Screw_Terminal_01x02, GoG_Library:TerminalBlock_WJ126V-5.0-2P_1x02_P5.00mm, F.Cu at (212.0, 134.2)
- added J9: Conn_01x02, Connector_JST:JST_XH_B2B-XH-A_1x02_P2.50mm_Vertical, F.Cu at (185.0, 143.5)
- added L1: 2.2u, GoG_Library:MDA5030-2R2M, F.Cu at (268.5, 127.9)
- added L2: 3.9u, Inductor_SMD:L_Sunlord_SWPA4030S, F.Cu at (169.3, 163.2)
- added L3: 4.7u, Inductor_SMD:L_Sunlord_SWPA4030S, F.Cu at (202.7, 153.5)
- added Q1: Q_PMOS, Package_TO_SOT_SMD:SOT-23, F.Cu at (249.5, 137.9)
- added Q2: Q_NMOS, Package_TO_SOT_SMD:SOT-23, F.Cu at (249.5, 142.5)
- added Q3: Q_NMOS, Package_TO_SOT_SMD:SOT-23, F.Cu at (249.5, 147.1)
- added Q4: Q_NMOS, Package_TO_SOT_SMD:SOT-23, F.Cu at (249.5, 151.8)
- added Q5: Q_NMOS, Package_TO_SOT_SMD:SOT-23, F.Cu at (249.5, 156.4)
- added R1: 1k, Resistor_SMD:R_0603_1608Metric, F.Cu at (192.8, 101.8)
- added R10: 1k, Resistor_SMD:R_0603_1608Metric, F.Cu at (131.8, 132.0)
- added R11: 470, Resistor_SMD:R_0603_1608Metric, F.Cu at (110.0, 123.5)
- added R12: 470, Resistor_SMD:R_0603_1608Metric, F.Cu at (110.0, 120.5)
- added R13: 22, Resistor_SMD:R_0603_1608Metric, F.Cu at (131.0, 129.0)
- added R14: 22, Resistor_SMD:R_0603_1608Metric, F.Cu at (123.5, 120.0)
- added R15: 0, Resistor_SMD:R_1206_3216Metric, F.Cu at (243.7, 154.0)
- added R16: 300, Resistor_SMD:R_0603_1608Metric, F.Cu at (262.4, 128.2)
- added R17: 100k, Resistor_SMD:R_0402_1005Metric, F.Cu at (234.3, 140.2)
- added R18: 300, Resistor_SMD:R_0603_1608Metric, F.Cu at (262.4, 130.7)
- added R19: 10k, Resistor_SMD:R_0402_1005Metric, F.Cu at (234.3, 142.2)
- added R2: 10k, Resistor_SMD:R_0603_1608Metric, F.Cu at (223.2, 102.5)
- added R20: 2.2k, Resistor_SMD:R_0402_1005Metric, F.Cu at (234.3, 144.2)
- added R21: 100, Resistor_SMD:R_0402_1005Metric, F.Cu at (237.2, 140.2)
- added R22: 5.1k, Resistor_SMD:R_0402_1005Metric, F.Cu at (237.2, 142.2)
- added R23: 120k, Resistor_SMD:R_0402_1005Metric, F.Cu at (237.2, 144.2)
- added R24: 8.2k, Resistor_SMD:R_0402_1005Metric, F.Cu at (240.2, 140.2)
- added R25: 30k, Resistor_SMD:R_0402_1005Metric, F.Cu at (240.2, 142.2)
- added R26: 100k, Resistor_SMD:R_0402_1005Metric, F.Cu at (240.2, 144.2)
- added R3: 10k, Resistor_SMD:R_0603_1608Metric, F.Cu at (142.2, 91.0)
- added R4: 4.7k, Resistor_SMD:R_0603_1608Metric, F.Cu at (222.9, 93.0)
- added R5: 4.7k, Resistor_SMD:R_0603_1608Metric, F.Cu at (222.9, 95.5)
- added R6: 10k, Resistor_SMD:R_0603_1608Metric, F.Cu at (186.8, 85.5)
- added R7: 5k1, Resistor_SMD:R_0603_1608Metric, F.Cu at (205.5, 114.0)
- added R8: 5k1, Resistor_SMD:R_0603_1608Metric, F.Cu at (205.5, 110.5)
- added R9: 0, Resistor_SMD:R_0805_2012Metric_Pad1.20x1.40mm_HandSolder, F.Cu at (114.5, 95.0)
- added REF**: MountingHole_3.2mm_M3, MountingHole:MountingHole_3.2mm_M3, F.Cu at (103.0, 87.5)
- added REF**: MountingHole_3.2mm_M3, MountingHole:MountingHole_3.2mm_M3, F.Cu at (213.0, 143.5)
- added REF**: MountingHole_3.2mm_M3, MountingHole:MountingHole_3.2mm_M3, F.Cu at (103.0, 143.5)
- added REF**: MountingHole_3.2mm_M3, MountingHole:MountingHole_3.2mm_M3, F.Cu at (213.0, 87.5)
- added SW1: SW_Omron_B3FS, Button_Switch_SMD:SW_SPST_Omron_B3FS-100xP, F.Cu at (181.3, 106.8)
- added SW2: SW_Omron_B3FS, Button_Switch_SMD:SW_SPST_Omron_B3FS-100xP, F.Cu at (181.3, 98.0)
- added TH1: 10k, GoG_Library:Thermistor NTC, F.Cu at (266.1, 142.8)
- added TP1: TestPoint_2Pole, Connector_PinHeader_2.54mm:PinHeader_2x01_P2.54mm_Vertical, F.Cu at (254.3, 155.7)
- added TP10: TestPoint, GoG_Library:TestPoint_Pad_D1.5mm_JLCPCB, F.Cu at (238.2, 119.7)
- added TP11: TestPoint, GoG_Library:TestPoint_Pad_D1.5mm_JLCPCB, F.Cu at (238.2, 123.3)
- added TP12: TestPoint, GoG_Library:TestPoint_Pad_D1.5mm_JLCPCB, F.Cu at (238.2, 126.8)
- added TP13: TestPoint, GoG_Library:TestPoint_Pad_D1.5mm_JLCPCB, F.Cu at (238.2, 130.4)
- added TP14: TestPoint, GoG_Library:TestPoint_Pad_D1.5mm_JLCPCB, F.Cu at (238.2, 133.9)
- added TP15: TestPoint, GoG_Library:TestPoint_Pad_D1.5mm_JLCPCB, F.Cu at (238.2, 137.5)
- added TP16: TestPoint, GoG_Library:TestPoint_Pad_D1.5mm_JLCPCB, F.Cu at (241.8, 116.2)
- added TP17: TestPoint, GoG_Library:TestPoint_Pad_D1.5mm_JLCPCB, F.Cu at (241.8, 119.7)
- added TP18: TestPoint, GoG_Library:TestPoint_Pad_D1.5mm_JLCPCB, F.Cu at (241.8, 123.3)
- added TP19: TestPoint, GoG_Library:TestPoint_Pad_D1.5mm_JLCPCB, F.Cu at (241.8, 126.8)
- added TP2: TestPoint, GoG_Library:TestPoint_Pad_D1.5mm_JLCPCB, F.Cu at (234.7, 116.2)
- added TP20: TestPoint, GoG_Library:TestPoint_Pad_D1.5mm_JLCPCB, F.Cu at (241.8, 130.4)
- added TP21: TestPoint, GoG_Library:TestPoint_Pad_D1.5mm_JLCPCB, F.Cu at (241.8, 133.9)
- added TP22: TestPoint, GoG_Library:TestPoint_Pad_D1.5mm_JLCPCB, F.Cu at (241.8, 137.5)
- added TP23: TestPoint, GoG_Library:TestPoint_Pad_D1.5mm_JLCPCB, F.Cu at (245.3, 116.2)
- added TP24: TestPoint, GoG_Library:TestPoint_Pad_D1.5mm_JLCPCB, F.Cu at (245.3, 119.7)
- added TP25: TestPoint, GoG_Library:TestPoint_Pad_D1.5mm_JLCPCB, F.Cu at (245.3, 123.3)
- added TP26: TestPoint, GoG_Library:TestPoint_Pad_D1.5mm_JLCPCB, F.Cu at (245.3, 126.8)
- added TP27: TestPoint, GoG_Library:TestPoint_Pad_D1.5mm_JLCPCB, F.Cu at (245.3, 130.4)
- added TP28: TestPoint, GoG_Library:TestPoint_Pad_D1.5mm_JLCPCB, F.Cu at (162.3, 155.7)
- added TP29: TestPoint, GoG_Library:TestPoint_Pad_D1.5mm_JLCPCB, F.Cu at (191.7, 154.0)
- added TP3: TestPoint, GoG_Library:TestPoint_Pad_D1.5mm_JLCPCB, F.Cu at (234.7, 119.7)
- added TP4: TestPoint, GoG_Library:TestPoint_Pad_D1.5mm_JLCPCB, F.Cu at (234.7, 123.3)
- added TP5: TestPoint, GoG_Library:TestPoint_Pad_D1.5mm_JLCPCB, F.Cu at (234.7, 126.8)
- added TP6: TestPoint, GoG_Library:TestPoint_Pad_D1.5mm_JLCPCB, F.Cu at (234.7, 130.4)
- added TP7: TestPoint, GoG_Library:TestPoint_Pad_D1.5mm_JLCPCB, F.Cu at (234.7, 133.9)
- added TP8: TestPoint, GoG_Library:TestPoint_Pad_D1.5mm_JLCPCB, F.Cu at (234.7, 137.5)
- added TP9: TestPoint, GoG_Library:TestPoint_Pad_D1.5mm_JLCPCB, F.Cu at (238.2, 116.2)
- added TP_DIO1: TestPoint, GoG_Library:TestPoint_Pad_D1.5mm_JLCPCB, F.Cu at (122.5, 113.5)
- added TP_RESET1: TestPoint, GoG_Library:TestPoint_Pad_D1.5mm_JLCPCB, F.Cu at (143.0, 96.5)
- added TP_VCC_Lora1: TestPoint, GoG_Library:TestPoint_Pad_D1.5mm_JLCPCB, F.Cu at (117.0, 103.0)
- added U1: ESP32-C3-WROOM-02, RF_Module:ESP32-C3-WROOM-02, F.Cu at (198.9, 90.6)
- added U2: USBLC6-2SC6, Package_TO_SOT_SMD:SOT-23-6, F.Cu at (203.0, 103.5)
- added U3: RFM95W-868S2, RF_Module:HOPERF_RFM9XW_SMD, F.Cu at (130.0, 102.0)
- added U4: SAM-M8Q, RF_GPS:ublox_SAM-M8Q, F.Cu at (120.5, 129.9)
- added U5: BQ25798RQMR, BQ25798RQMR:IC_BQ25798RQMR, F.Cu at (192.0, 134.0)
- added U6: AP63203WU, Package_TO_SOT_SMD:TSOT-23-6, F.Cu at (161.8, 162.9)
- added U7: AP63205WU, Package_TO_SOT_SMD:TSOT-23-6, F.Cu at (191.4, 159.4)
Other:
- board outline added: 118 x 64 mm
