File: hardware/ESP32.kicad_sch (KiCad schematic)
At the start: 20 parts, among them J1 USB_C_Receptacle_USB2.0_16P, J10 Conn_01x04_Pin, J11 Conn_01x02_Pin, J9 Conn_01x02_Pin, SW1 SW_Omron_B3FS, SW2 SW_Omron_B3FS, U2 ESP32-C3-WROOM-02, U8 USBLC6-2SC6

Commit message: Setup PCB design parameters
Connections:
- net D+ renamed USB_D+
- net D- renamed USB_D-
Changed lines of the file:
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@@
 	(wire
 		(pts
-			(xy 191.77 78.74) (xy 198.12 78.74)
+			(xy 195.58 78.74) (xy 198.12 78.74)
 		)
 		(stroke
@@
 	(wire
 		(pts
-			(xy 191.77 81.28) (xy 198.12 81.28)
+			(xy 195.58 81.28) (xy 198.12 81.28)
 		)
 		(stroke
@@
 		)
 	)
-	(label "D-"
-		(at 191.77 78.74 180)
+	(label "USB_D-"
+		(at 195.58 78.74 180)
 		(effects
 			(font
@@
 		)
 	)
-	(label "D-"
+	(label "USB_D-"
 		(at 134.62 102.87 0)
 		(effects
@@
 		)
 	)
-	(label "D+"
-		(at 191.77 81.28 180)
+	(label "USB_D+"
+		(at 195.58 81.28 180)
 		(effects
 			(font
@@
 		)
 	)
-	(label "D+"
+	(label "USB_D+"
 		(at 134.62 105.41 0)
 		(effects

Commit message: Fix schematic components annotations
Parts:
- renumbered D7 to D1, J9 to J2, J10 to J3, J11 to J4, R19 to R1, R6 to R4, R7 to R5, R1 to R6, R4 to R7, R5 to R8, U2 to U1, U8 to U2
Changed lines of the file:
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@@
 		(dnp no)
 		(fields_autoplaced yes)
-		(property "Reference" "R4"
+		(property "Reference" "R7"
 			(at 72.39 96.5199 0)
 			(effects
@@
 			(project "GOG"
 				(path "/5b969f6e-a36e-432b-8f00-b2d6a515a877/36e0c9fb-3d9d-4ab1-92fc-4f7433c1320d"
-					(reference "R4")
+					(reference "R7")
 					(unit 1)
 				)
@@
 		(dnp no)
 		(fields_autoplaced yes)
-		(property "Reference" "U2"
+		(property "Reference" "U1"
 			(at 215.5033 38.1 0)
 			(effects
@@
 			(project ""
 				(path "/5b969f6e-a36e-432b-8f00-b2d6a515a877/36e0c9fb-3d9d-4ab1-92fc-4f7433c1320d"
-					(reference "U2")
+					(reference "U1")
 					(unit 1)
 				)
@@
 		(dnp no)
 		(fields_autoplaced yes)
-		(property "Reference" "#PWR02"
+		(property "Reference" "#PWR010"
 			(at 204.47 114.3 0)
 			(effects
@@
 			(project "GOG"
 				(path "/5b969f6e-a36e-432b-8f00-b2d6a515a877/36e0c9fb-3d9d-4ab1-92fc-4f7433c1320d"
-					(reference "#PWR02")
+					(reference "#PWR010")
 					(unit 1)
 				)
@@
 		(on_board yes)
 		(dnp no)
-		(property "Reference" "R6"
+		(property "Reference" "R4"
 			(at 187.96 38.1 0)
 			(effects
@@
 			(project "GOG"
 				(path "/5b969f6e-a36e-432b-8f00-b2d6a515a877/36e0c9fb-3d9d-4ab1-92fc-4f7433c1320d"
-					(reference "R6")
+					(reference "R4")
 					(unit 1)
 				)
@@
 		(on_board yes)
 		(dnp no)
-		(property "Reference" "J10"
+		(property "Reference" "J3"
 			(at 157.48 137.16 0)
 			(effects
@@
 			(project ""
 				(path "/5b969f6e-a36e-432b-8f00-b2d6a515a877/36e0c9fb-3d9d-4ab1-92fc-4f7433c1320d"
-					(reference "J10")
+					(reference "J3")
 					(unit 1)
 				)
@@
 		(on_board yes)
 		(dnp no)
-		(property "Reference" "J11"
+		(property "Reference" "J4"
 			(at 157.48 152.4 0)
 			(effects
@@
 			(project "GOG"
 				(path "/5b969f6e-a36e-432b-8f00-b2d6a515a877/36e0c9fb-3d9d-4ab1-92fc-4f7433c1320d"
-					(reference "J11")
+					(reference "J4")
 					(unit 1)
 				)
@@
 		(dnp no)
 		(fields_autoplaced yes)
-		(property "Reference" "#PWR037"
+		(property "Reference" "#PWR01"
 			(at 88.9 58.42 0)
 			(effects
@@
 			(project "GOG"
 				(path "/5b969f6e-a36e-432b-8f00-b2d6a515a877/36e0c9fb-3d9d-4ab1-92fc-4f7433c1320d"
-					(reference "#PWR037")
+					(reference "#PWR01")
 					(unit 1)
 				)
@@
 		(dnp no)
 		(fields_autoplaced yes)
-		(property "Reference" "R1"
+		(property "Reference" "R6"
 			(at 149.86 39.3699 0)
 			(effects
@@
 			(project "GOG"
 				(path "/5b969f6e-a36e-432b-8f00-b2d6a515a877/36e0c9fb-3d9d-4ab1-92fc-4f7433c1320d"
-					(reference "R1")
+					(reference "R6")
 					(unit 1)
 				)
@@
 		(dnp no)
 		(fields_autoplaced yes)
-		(property "Reference" "#PWR04"
+		(property "Reference" "#PWR06"
 			(at 204.47 102.87 0)
 			(effects
@@
 			(project "GOG"
 				(path "/5b969f6e-a36e-432b-8f00-b2d6a515a877/36e0c9fb-3d9d-4ab1-92fc-4f7433c1320d"
-					(reference "#PWR04")
+					(reference "#PWR06")
 					(unit 1)
 				)
@@
 		(dnp no)
 		(fields_autoplaced yes)
-		(property "Reference" "#PWR03"
+		(property "Reference" "#PWR02"
 			(at 129.54 67.31 0)
 			(effects
@@
 			(project "GOG"
 				(path "/5b969f6e-a36e-432b-8f00-b2d6a515a877/36e0c9fb-3d9d-4ab1-92fc-4f7433c1320d"
-					(reference "#PWR03")
+					(reference "#PWR02")
 					(unit 1)
 				)
@@
 		(dnp no)
 		(fields_autoplaced yes)
-		(property "Reference" "#PWR012"
+		(property "Reference" "#PWR09"
 			(at 124.46 119.38 0)
 			(effects
@@
 			(project "GOG"
 				(path "/5b969f6e-a36e-432b-8f00-b2d6a515a877/36e0c9fb-3d9d-4ab1-92fc-4f7433c1320d"
-					(reference "#PWR012")
+					(reference "#PWR09")
 					(unit 1)
 				)
@@
 		(on_board yes)
 		(dnp no)
-		(property "Reference" "J9"
+		(property "Reference" "J2"
 			(at 157.48 127 0)
 			(effects
@@
 			(project ""
 				(path "/5b969f6e-a36e-432b-8f00-b2d6a515a877/36e0c9fb-3d9d-4ab1-92fc-4f7433c1320d"
-					(reference "J9")
+					(reference "J2")
 					(unit 1)
 				)
@@
 		(dnp no)
 		(fields_autoplaced yes)
-		(property "Reference" "D7"
+		(property "Reference" "D1"
 			(at 92.71 46.0374 90)
 			(effects
@@
 			(project "GOG"
 				(path "/5b969f6e-a36e-432b-8f00-b2d6a515a877/36e0c9fb-3d9d-4ab1-92fc-4f7433c1320d"
-					(reference "D7")
+					(reference "D1")
 					(unit 1)
 				)
@@
 		(dnp no)
 		(fields_autoplaced yes)
-		(property "Reference" "U8"
+		(property "Reference" "U2"
 			(at 126.1111 95.25 0)
 			(effects
@@
 			(project ""
 				(path "/5b969f6e-a36e-432b-8f00-b2d6a515a877/36e0c9fb-3d9d-4ab1-92fc-4f7433c1320d"
-					(reference "U8")
+					(reference "U2")
 					(unit 1)
 				)
@@
 		(dnp no)
 		(fields_autoplaced yes)
-		(property "Reference" "#PWR010"
+		(property "Reference" "#PWR07"
 			(at 69.85 111.76 0)
 			(effects
@@
 			(project "GOG"
 				(path "/5b969f6e-a36e-432b-8f00-b2d6a515a877/36e0c9fb-3d9d-4ab1-92fc-4f7433c1320d"
-					(reference "#PWR010")
+					(reference "#PWR07")
 					(unit 1)
 				)
@@
 		(dnp no)
 		(fields_autoplaced yes)
-		(property "Reference" "R5"
+		(property "Reference" "R8"
 			(at 80.01 96.5199 0)
 			(effects
@@
 			(project "GOG"
 				(path "/5b969f6e-a36e-432b-8f00-b2d6a515a877/36e0c9fb-3d9d-4ab1-92fc-4f7433c1320d"
-					(reference "R5")
+					(reference "R8")
 					(unit 1)
 				)
@@
 		(dnp no)
 		(fields_autoplaced yes)
-		(property "Reference" "#PWR01"
+		(property "Reference" "#PWR05"
 			(at 213.36 96.52 0)
 			(effects
@@
 			(project "GOG"
 				(path "/5b969f6e-a36e-432b-8f00-b2d6a515a877/36e0c9fb-3d9d-4ab1-92fc-4f7433c1320d"
-					(reference "#PWR01")
+					(reference "#PWR05")
 					(unit 1)
 				)
@@
 		(dnp no)
 		(fields_autoplaced yes)
-		(property "Reference" "#PWR016"
+		(property "Reference" "#PWR04"
 			(at 31.75 87.63 0)
 			(effects
@@
 			(project "GOG"
 				(path "/5b969f6e-a36e-432b-8f00-b2d6a515a877/36e0c9fb-3d9d-4ab1-92fc-4f7433c1320d"
-					(reference "#PWR016")
+					(reference "#PWR04")
 					(unit 1)
 				)
@@
 		(dnp no)
 		(fields_autoplaced yes)
-		(property "Reference" "#PWR015"
+		(property "Reference" "#PWR03"
 			(at 24.13 87.63 0)
 			(effects
@@
 			(project "GOG"
 				(path "/5b969f6e-a36e-432b-8f00-b2d6a515a877/36e0c9fb-3d9d-4ab1-92fc-4f7433c1320d"
-					(reference "#PWR015")
+					(reference "#PWR03")
 					(unit 1)
 				)
@@
 		(on_board yes)
 		(dnp no)
-		(property "Reference" "R7"
+		(property "Reference" "R5"
 			(at 195.58 38.1 0)
 			(effects
@@
 			(project "GOG"
 				(path "/5b969f6e-a36e-432b-8f00-b2d6a515a877/36e0c9fb-3d9d-4ab1-92fc-4f7433c1320d"
-					(reference "R7")
+					(reference "R5")
 					(unit 1)
 				)
@@
 		(dnp no)
 		(fields_autoplaced yes)
-		(property "Reference" "#PWR011"
+		(property "Reference" "#PWR08"
 			(at 77.47 111.76 0)
 			(effects
@@
 			(project "GOG"
 				(path "/5b969f6e-a36e-432b-8f00-b2d6a515a877/36e0c9fb-3d9d-4ab1-92fc-4f7433c1320d"
-					(reference "#PWR011")
+					(reference "#PWR08")
 					(unit 1)
 				)
@@
 		(dnp no)
 		(fields_autoplaced yes)
-		(property "Reference" "R19"
+		(property "Reference" "R1"
 			(at 91.44 36.8299 0)
 			(effects
@@
 			(project "GOG"
 				(path "/5b969f6e-a36e-432b-8f00-b2d6a515a877/36e0c9fb-3d9d-4ab1-92fc-4f7433c1320d"
-					(reference "R19")
-					(unit 1)
-				)
+					(reference "R1")
+					(unit 1)
+				)
