File: hardware/Power.kicad_sch (KiCad schematic)
At the start: 90 parts, among them J5 Screw_Terminal_01x02, J6 Conn_01x04, J7 Conn_01x02, J8 Conn_01x02, Q1 Q_NMOS, Q2 Q_NMOS, Q3 Q_NMOS, Q4 Q_NMOS, Q5 Q_PMOS, U1 AP63203WU, U3 AP63205WU, U5 BQ25798RQMR

Commit message: Fix schematic components annotations
Parts:
- renumbered C11 to C10, C12 to C11, C13 to C12, C5 to C13, C6 to C14, C7 to C15, C14 to C16, C9 to C17, C4 to C18, C15 to C19, C16 to C20, C17 to C21, C18 to C22, C19 to C23, C20 to C24, C21 to C25, C22 to C26, C23 to C27, C24 to C28, C28 to C29, C25 to C30, C26 to C31, C27 to C32, C32 to C33, C29 to C34, C30 to C35, C31 to C36, C10 to C9, D5 to D3, D3 to D4, D2 to D5, D4 to D6, J6 to J10, J7 to J11, J5 to J8, J8 to J9, Q5 to Q1, Q3 to Q2, Q4 to Q3, Q1 to Q4, Q2 to Q5, R22 to R15, R11 to R16, R20 to R17, R12 to R18, R23 to R19, R10 to R20, R18 to R21, R16 to R22, R14 to R23, R13 to R24, R17 to R25, R15 to R26, TP29 to TP1, TP18 to TP11, TP19 to TP12, TP7 to TP13, TP3 to TP14, TP20 to TP15, TP21 to TP16, TP22 to TP17, TP11 to TP18, TP23 to TP19, TP12 to TP20, TP14 to TP21, TP13 to TP22, TP24 to TP23, TP15 to TP24, TP16 to TP26, TP26 to TP27, TP27 to TP28, TP28 to TP29, TP5 to TP3, TP1 to TP4, TP6 to TP5, TP4 to TP6, TP17 to TP7, TP9 to TP8, TP8 to TP9, U1 to U6, U3 to U7

Commit message: Fix all ERC errors
Parts:
- U5: footprint RQM0029A-MFG -> BQ25798RQMR:RQM0029A-MFG
Connections:
- net +3V3 renamed 3.3V
- net +5V renamed 5V
- net V_REGN renamed REGN
Other:
- moved on the sheet: C10, C11, C12, J8, J9, TP10, TP17, TP7

Commit message: Fix several DRC errors & add all 3D models
Parts:
- Q1: symbol Device:Q_PMOS -> AO3415:AO3415
- Q2, Q3, Q4, Q5: symbol Device:Q_NMOS -> AO3400:AO3400
- TP10, TP11, TP12, TP13, TP14, TP15, TP16, TP17, TP18, TP19, TP2, TP20, TP21, TP22, TP23, TP24, TP25, TP26, TP27, TP28, TP29, TP3, TP4, TP5, TP6, TP7, TP8, TP9: footprint TestPoint:TestPoint_Pad_D1.5mm -> GoG_Library:TestPoint_Pad_D1.5mm_JLCPCB
- U5: footprint BQ25798RQMR:RQM0029A-MFG -> BQ25798RQMR:IC_BQ25798RQMR
Connections:
- net VBUS: now also Q4.3 (D); no longer Q4.D
- net at D4.2 (A), TP5.1: now also Q2.2 (S), Q3.2 (S); no longer Q2.S, Q3.S
- net at C13.1, C14.1, C15.1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: now also Q3.3 (D), Q5.3 (D); no longer Q3.D, Q5.D
- net at D3.2 (A), R17.2, TP4.1: now also Q1.1 (G); no longer Q1.G
- net at C8.1, D3.1 (K), TP2.1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: now also Q1.2 (S), Q2.3 (D); no longer Q1.S, Q2.D
- net at D4.1 (K), R16.1, TP3.1: now also Q2.1 (G), Q3.1 (G); no longer Q2.G, Q3.G
- net at D5.1 (K), R18.1, TP13.1: now also Q4.1 (G), Q5.1 (G); no longer Q4.G, Q5.G
- net at D5.2 (A), TP9.1: now also Q4.2 (S), Q5.2 (S); no longer Q4.S, Q5.S
- net at R15.1, TP1.2: now also Q1.3 (D); no longer Q1.D
Changed lines of the file:
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@@
 			)
 		)
-		(property "Footprint" "TestPoint:TestPoint_Pad_D1.5mm"
+		(property "Footprint" "GoG_Library:TestPoint_Pad_D1.5mm_JLCPCB"
 			(at 185.42 86.36 0)
 			(effects
@@
 			)
 		)
-		(property "Footprint" "TestPoint:TestPoint_Pad_D1.5mm"
+		(property "Footprint" "GoG_Library:TestPoint_Pad_D1.5mm_JLCPCB"
 			(at 99.06 40.64 0)
 			(effects
@@
 			)
 		)
-		(property "Footprint" "TestPoint:TestPoint_Pad_D1.5mm"
+		(property "Footprint" "GoG_Library:TestPoint_Pad_D1.5mm_JLCPCB"
 			(at 104.14 85.09 0)
 			(effects
@@
 	)
 	(symbol
-		(lib_id "Device:Q_NMOS")
+		(lib_id "AO3400:AO3400")
 		(at 111.76 53.34 270)
 		(mirror x)
@@
 			)
 		)
-		(property "Description" "AO3400 N-Channel 1.5W 1.05nF 30V 28mΩ@10V 1.4V@250uA"
+		(property "Description" "N-MOSFET transistor"
 			(at 111.76 53.34 0)
 			(effects
@@
 			)
 		)
-		(pin "D"
+		(pin "3"
 		)
-		(pin "S"
+		(pin "1"
 		)
-		(pin "G"
+		(pin "2"
 		)
 		(instances
@@
 			)
 		)
-		(property "Footprint" "TestPoint:TestPoint_Pad_D1.5mm"
+		(property "Footprint" "GoG_Library:TestPoint_Pad_D1.5mm_JLCPCB"
 			(at 104.14 54.61 0)
 			(effects
@@
 			)
 		)
-		(property "Footprint" "TestPoint:TestPoint_Pad_D1.5mm"
+		(property "Footprint" "GoG_Library:TestPoint_Pad_D1.5mm_JLCPCB"
 			(at 184.15 49.53 0)
 			(effects
@@
 			)
 		)
-		(property "Footprint" "TestPoint:TestPoint_Pad_D1.5mm"
+		(property "Footprint" "GoG_Library:TestPoint_Pad_D1.5mm_JLCPCB"
 			(at 144.78 44.45 0)
 			(effects
@@
 			)
 		)
-		(property "Footprint" "TestPoint:TestPoint_Pad_D1.5mm"
+		(property "Footprint" "GoG_Library:TestPoint_Pad_D1.5mm_JLCPCB"
 			(at 133.35 90.17 0)
 			(effects
@@
 			)
 		)
-		(property "Footprint" "TestPoint:TestPoint_Pad_D1.5mm"
+		(property "Footprint" "GoG_Library:TestPoint_Pad_D1.5mm_JLCPCB"
 			(at 144.78 83.82 0)
 			(effects
@@
 			)
 		)
-		(property "Footprint" "TestPoint:TestPoint_Pad_D1.5mm"
+		(property "Footprint" "GoG_Library:TestPoint_Pad_D1.5mm_JLCPCB"
 			(at 185.42 91.44 0)
 			(effects
@@
 			)
 		)
-		(property "Footprint" "TestPoint:TestPoint_Pad_D1.5mm"
+		(property "Footprint" "GoG_Library:TestPoint_Pad_D1.5mm_JLCPCB"
 			(at 196.85 41.91 0)
 			(effects
@@
 			)
 		)
-		(property "Footprint" "TestPoint:TestPoint_Pad_D1.5mm"
+		(property "Footprint" "GoG_Library:TestPoint_Pad_D1.5mm_JLCPCB"
 			(at 147.32 54.61 0)
 			(effects
@@
 			)
 		)
-		(property "Footprint" "TestPoint:TestPoint_Pad_D1.5mm"
+		(property "Footprint" "GoG_Library:TestPoint_Pad_D1.5mm_JLCPCB"
 			(at 133.35 93.98 0)
 			(effects
@@
 			)
 		)
-		(property "Footprint" "TestPoint:TestPoint_Pad_D1.5mm"
+		(property "Footprint" "GoG_Library:TestPoint_Pad_D1.5mm_JLCPCB"
 			(at 93.98 29.21 0)
 			(effects
@@
 	)
 	(symbol
-		(lib_id "Device:Q_PMOS")
+		(lib_id "AO3415:AO3415")
 		(at 71.12 31.75 90)
 		(unit 1)
@@
 			)
 		)
-		(property "Description" "AO3415 P-Channel 1.39W 115pF 20V 30mΩ@4.5V SOT-23 MOSFET"
+		(property "Description" "P-MOSFET transistor"
 			(at 71.12 31.75 0)
 			(effects
@@
 			)
 		)
-		(pin "D"
+		(pin "1"
 		)
-		(pin "G"
+		(pin "3"
 		)
-		(pin "S"
+		(pin "2"
 		)
 		(instances
@@
 			)
 		)
-		(property "Footprint" "TestPoint:TestPoint_Pad_D1.5mm"
+		(property "Footprint" "GoG_Library:TestPoint_Pad_D1.5mm_JLCPCB"
 			(at 209.55 63.5 0)
 			(effects
@@
 			)
 		)
-		(property "Footprint" "TestPoint:TestPoint_Pad_D1.5mm"
+		(property "Footprint" "GoG_Library:TestPoint_Pad_D1.5mm_JLCPCB"
 			(at 82.55 142.24 0)
 			(effects
@@
 			)
 		)
-		(property "Footprint" "BQ25798RQMR:RQM0029A-MFG"
+		(property "Footprint" "BQ25798RQMR:IC_BQ25798RQMR"
 			(at 146.05 43.18 0)
 			(effects
@@
 	)
 	(symbol
-		(lib_id "Device:Q_NMOS")
+		(lib_id "AO3400:AO3400")
 		(at 96.52 53.34 90)
 		(unit 1)
@@
 			)
 		)
-		(property "Description" "AO3400 N-Channel 1.5W 1.05nF 30V 28mΩ@10V 1.4V@250uA"
+		(property "Description" "N-MOSFET transistor"
 			(at 96.52 53.34 0)
 			(effects
@@
 			)
 		)
-		(pin "D"
+		(pin "3"
 		)
-		(pin "S"
+		(pin "1"
 		)
-		(pin "G"
+		(pin "2"
 		)
 		(instances
@@
 			)
 		)
-		(property "Footprint" "TestPoint:TestPoint_Pad_D1.5mm"
+		(property "Footprint" "GoG_Library:TestPoint_Pad_D1.5mm_JLCPCB"
 			(at 184.15 64.77 0)
 			(effects
@@
 			)
 		)
-		(property "Footprint" "TestPoint:TestPoint_Pad_D1.5mm"
+		(property "Footprint" "GoG_Library:TestPoint_Pad_D1.5mm_JLCPCB"
 			(at 93.98 62.23 0)
 			(effects
@@
 	)
 	(symbol
-		(lib_id "Device:Q_NMOS")
+		(lib_id "AO3400:AO3400")
 		(at 96.52 38.1 90)
 		(mirror x)
@@
 			)
 		)
-		(property "Description" "AO3400 N-Channel 1.5W 1.05nF 30V 28mΩ@10V 1.4V@250uA"
+		(property "Description" "N-MOSFET transistor"
 			(at 96.52 38.1 0)
 			(effects
@@
 			)
 		)
-		(pin "D"
+		(pin "2"
 		)
-		(pin "S"
+		(pin "3"
 		)
-		(pin "G"
+		(pin "1"
 		)
 		(instances
@@
 			)
 		)
-		(property "Footprint" "TestPoint:TestPoint_Pad_D1.5mm"
+		(property "Footprint" "GoG_Library:TestPoint_Pad_D1.5mm_JLCPCB"
 			(at 185.42 82.55 0)
 			(effects
@@
 			)
 		)
-		(property "Footprint" "TestPoint:TestPoint_Pad_D1.5mm"
+		(property "Footprint" "GoG_Library:TestPoint_Pad_D1.5mm_JLCPCB"
 			(at 69.85 31.75 0)
 			(effects
@@
 			)
 		)
-		(property "Footprint" "TestPoint:TestPoint_Pad_D1.5mm"
+		(property "Footprint" "GoG_Library:TestPoint_Pad_D1.5mm_JLCPCB"
 			(at 133.35 91.44 0)
 			(effects
@@
 			)
 		)
-		(property "Footprint" "TestPoint:TestPoint_Pad_D1.5mm"
+		(property "Footprint" "GoG_Library:TestPoint_Pad_D1.5mm_JLCPCB"
 			(at 222.25 81.28 0)
 			(effects
@@
 			)
 		)
-		(property "Footprint" "TestPoint:TestPoint_Pad_D1.5mm"
+		(property "Footprint" "GoG_Library:TestPoint_Pad_D1.5mm_JLCPCB"
 			(at 83.82 176.53 0)
 			(effects
@@
 			)
 		)
-		(property "Footprint" "TestPoint:TestPoint_Pad_D1.5mm"
+		(property "Footprint" "GoG_Library:TestPoint_Pad_D1.5mm_JLCPCB"
 			(at 144.78 80.01 0)
 			(effects
@@
 			)
 		)
-		(property "Footprint" "TestPoint:TestPoint_Pad_D1.5mm"
+		(property "Footprint" "GoG_Library:TestPoint_Pad_D1.5mm_JLCPCB"
 			(at 142.24 40.64 0)
 			(effects
@@
 	)
 	(symbol
-		(lib_id "Device:Q_NMOS")
+		(lib_id "AO3400:AO3400")
 		(at 111.76 38.1 270)
 		(unit 1)
@@
 			)
 		)
-		(property "Description" "AO3400 N-Channel 1.5W 1.05nF 30V 28mΩ@10V 1.4V@250uA"
+		(property "Description" "N-MOSFET transistor"
 			(at 111.76 38.1 0)
 			(effects
@@
 			)
 		)
-		(pin "D"
+		(pin "3"
 		)
-		(pin "S"
+		(pin "1"
 		)
-		(pin "G"
+		(pin "2"
 		)
 		(instances
@@
 			)
 		)
-		(property "Footprint" "TestPoint:TestPoint_Pad_D1.5mm"
+		(property "Footprint" "GoG_Library:TestPoint_Pad_D1.5mm_JLCPCB"
 			(at 209.55 73.66 0)
 			(effects
@@
 			)
 		)
-		(property "Footprint" "TestPoint:TestPoint_Pad_D1.5mm"
+		(property "Footprint" "GoG_Library:TestPoint_Pad_D1.5mm_JLCPCB"
 			(at 185.42 96.52 0)
 			(effects
@@
 			)
 		)
-		(property "Footprint" "TestPoint:TestPoint_Pad_D1.5mm"
+		(property "Footprint" "GoG_Library:TestPoint_Pad_D1.5mm_JLCPCB"
 			(at 104.14 26.67 0)
 			(effects
@@
 			)
 		)
-		(property "Footprint" "TestPoint:TestPoint_Pad_D1.5mm"
+		(property "Footprint" "GoG_Library:TestPoint_Pad_D1.5mm_JLCPCB"
 			(at 109.22 50.8 0)
 			(effects

Commit message: Finished battery manager placement
Parts:
- removed R15: 0, Resistor_SMD:R_1206_3216Metric, symbol Device:R
- removed TP1: TestPoint_2Pole, Connector_PinHeader_2.54mm:PinHeader_2x01_P2.54mm_Vertical, symbol Connector:TestPoint_2Pole
- removed TP11, TP16, TP19, TP23: TestPoint, GoG_Library:TestPoint_Pad_D1.5mm_JLCPCB, symbol Connector:TestPoint
- C15, C18, C20, C28, C8, C9: footprint Capacitor_SMD:C_0402_1005Metric -> GoG_Library:C_0402_1005Metric_JLCPCB
- C16, C19: footprint Capacitor_SMD:C_0603_1608Metric -> GoG_Library:C_0402_1005Metric_JLCPCB; JLCPCB Part # C113811 -> C107020; Package 0603 -> 0402
- R16: renamed from R17; footprint Resistor_SMD:R_0402_1005Metric -> GoG_Library:R_0402_1005Metric_JLCPCB
- R18: renamed from R19; footprint Resistor_SMD:R_0402_1005Metric -> GoG_Library:R_0402_1005Metric_JLCPCB
- R19: renamed from R20; footprint Resistor_SMD:R_0402_1005Metric -> GoG_Library:R_0402_1005Metric_JLCPCB
- R20: renamed from R21; footprint Resistor_SMD:R_0402_1005Metric -> GoG_Library:R_0402_1005Metric_JLCPCB
- R21: renamed from R22; footprint Resistor_SMD:R_0402_1005Metric -> GoG_Library:R_0402_1005Metric_JLCPCB
- R22: renamed from R23; footprint Resistor_SMD:R_0402_1005Metric -> GoG_Library:R_0402_1005Metric_JLCPCB
- R23: renamed from R24; footprint Resistor_SMD:R_0402_1005Metric -> GoG_Library:R_0402_1005Metric_JLCPCB
- R24: renamed from R25; footprint Resistor_SMD:R_0402_1005Metric -> GoG_Library:R_0402_1005Metric_JLCPCB
- R25: renamed from R26; footprint Resistor_SMD:R_0402_1005Metric -> GoG_Library:R_0402_1005Metric_JLCPCB
- renumbered R16 to R15, R18 to R17, TP2 to TP1, TP12 to TP10, TP13 to TP11, TP14 to TP12, TP15 to TP13, TP17 to TP14, TP18 to TP15, TP20 to TP16, TP21 to TP17, TP22 to TP18, TP24 to TP19, TP3 to TP2, TP25 to TP20, TP26 to TP21, TP27 to TP22, TP28 to TP23, TP29 to TP24, TP4 to TP3, TP5 to TP4, TP6 to TP5, TP7 to TP6, TP8 to TP7, TP9 to TP8, TP10 to TP9
Connections:
- net VSOL: now also Q1.3 (D)
Other:
- moved on the sheet: J8
