File: hardware/Lora_Module.kicad_sch (KiCad schematic)
At the start: 9 parts, among them J5 85201239, U3 RFM95W-868S2

Commit message: Finished battery manager placement
Parts:
- U3: footprint RF_Module:HOPERF_RFM9XW_SMD -> GoG_Library:HOPERF_RFM9XW_SMD
Changed lines of the file:
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@@
 			)
 		)
-		(property "Footprint" "RF_Module:HOPERF_RFM9XW_SMD"
+		(property "Footprint" "GoG_Library:HOPERF_RFM9XW_SMD"
 			(at 25.4 30.48 0)
 			(effects

Commit message: Finished optimal placement & adapted/fixed schematic
Parts:
- removed TP_VCC_Lora1: TestPoint, GoG_Library:TestPoint_Pad_D1.5mm_JLCPCB, symbol Connector:TestPoint
- renumbered TP_RESET1 to TP1, TP_DIO1 to TP2
Connections:
- net 3.3V: now also C4.1; no longer C4.2
- net GND: now also C4.2; no longer C4.1
Other:
- moved on the sheet: C4, TP1, TP2
Changed lines of the file:
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@@
-	)
-	(junction
-		(at 109.22 38.1)
-		(diameter 0)
-		(color 0 0 0 0)
 	)
 	(junction
@@
 	)
 	(junction
-		(at 109.22 50.8)
+		(at 165.1 64.77)
 		(diameter 0)
 		(color 0 0 0 0)
 	)
 	(junction
-		(at 165.1 64.77)
+		(at 97.79 44.45)
 		(diameter 0)
 		(color 0 0 0 0)
@@
 	(wire
 		(pts
-			(xy 81.28 87.63) (xy 95.25 87.63)
+			(xy 93.98 81.28) (xy 95.25 81.28)
 		)
 		(stroke
@@
 	(wire
 		(pts
-			(xy 124.46 92.71) (xy 125.73 92.71)
-		)
-		(stroke
-			(width 0)
-			(type default)
-		)
-	)
-	(wire
-		(pts
-			(xy 109.22 38.1) (xy 86.36 38.1)
+			(xy 109.22 44.45) (xy 97.79 44.45)
 		)
 		(stroke
@@
 	(wire
 		(pts
-			(xy 109.22 50.8) (xy 109.22 38.1)
+			(xy 97.79 44.45) (xy 92.71 44.45)
 		)
 		(stroke
@@
 	(wire
 		(pts
-			(xy 95.25 87.63) (xy 95.25 77.47)
-		)
-		(stroke
-			(width 0)
-			(type default)
-		)
-	)
-	(wire
-		(pts
-			(xy 125.73 92.71) (xy 125.73 82.55)
+			(xy 95.25 81.28) (xy 95.25 77.47)
+		)
+		(stroke
+			(width 0)
+			(type default)
+		)
+	)
+	(wire
+		(pts
+			(xy 125.73 81.28) (xy 125.73 82.55)
 		)
 		(stroke
@@
 	(wire
 		(pts
+			(xy 97.79 44.45) (xy 97.79 45.72)
+		)
+		(stroke
+			(width 0)
+			(type default)
+		)
+	)
+	(wire
+		(pts
 			(xy 81.28 67.31) (xy 96.52 67.31)
 		)
@@
 	(wire
 		(pts
-			(xy 127 38.1) (xy 116.84 38.1)
-		)
-		(stroke
-			(width 0)
-			(type default)
-		)
-	)
-	(wire
-		(pts
 			(xy 179.07 72.39) (xy 179.07 69.85)
 		)
@@
 	(wire
 		(pts
-			(xy 92.71 50.8) (xy 109.22 50.8)
-		)
-		(stroke
-			(width 0)
-			(type default)
-		)
-	)
-	(wire
-		(pts
 			(xy 111.76 91.44) (xy 111.76 95.25)
 		)
@@
 	(wire
 		(pts
-			(xy 109.22 59.69) (xy 109.22 50.8)
+			(xy 109.22 44.45) (xy 109.22 59.69)
 		)
 		(stroke
@@
 	(global_label "3.3V"
 		(shape input)
-		(at 86.36 38.1 180)
+		(at 92.71 44.45 180)
 		(fields_autoplaced yes)
 		(effects
@@
 		)
 		(property "Intersheetrefs" "${INTERSHEET_REFS}"
-			(at 79.2624 38.1 0)
+			(at 85.6124 44.45 0)
 			(effects
 				(font
@@
 	(symbol
 		(lib_id "Connector:TestPoint")
-		(at 124.46 92.71 0)
+		(at 125.73 81.28 0)
 		(unit 1)
 		(exclude_from_sim no)
@@
 		(dnp no)
 		(fields_autoplaced yes)
-		(property "Reference" "TP_DIO1"
-			(at 127 88.1379 0)
+		(property "Reference" "TP2"
+			(at 128.27 76.7079 0)
 			(effects
 				(font
@@
 		)
 		(property "Value" "TestPoint"
-			(at 127 90.6779 0)
+			(at 128.27 79.2479 0)
 			(effects
 				(font
@@
 				)
 				(justify left)
+				(hide yes)
 			)
 		)
 		(property "Footprint" "GoG_Library:TestPoint_Pad_D1.5mm_JLCPCB"
-			(at 129.54 92.71 0)
+			(at 130.81 81.28 0)
 			(effects
 				(font
@@
 		)
 		(property "Datasheet" "~"
-			(at 129.54 92.71 0)
+			(at 130.81 81.28 0)
 			(effects
 				(font
@@
 		)
 		(property "Description" "test point"
-			(at 124.46 92.71 0)
+			(at 125.73 81.28 0)
 			(effects
 				(font
@@
 			(project ""
 				(path "/5b969f6e-a36e-432b-8f00-b2d6a515a877/9db73a32-37a4-4249-8656-c1ba9b3afe01"
-					(reference "TP_DIO1")
+					(reference "TP2")
 					(unit 1)
 				)
@@
 	(symbol
 		(lib_id "Connector:TestPoint")
-		(at 81.28 87.63 0)
+		(at 93.98 81.28 90)
 		(unit 1)
 		(exclude_from_sim no)
@@
 		(on_board yes)
 		(dnp no)
-		(fields_autoplaced yes)
-		(property "Reference" "TP_RESET1"
-			(at 83.82 83.0579 0)
+		(property "Reference" "TP1"
+			(at 86.36 81.28 90)
+			(effects
+				(font
+					(size 1.27 1.27)
+				)
+			)
+		)
+		(property "Value" "TestPoint"
+			(at 91.9479 78.74 0)
 			(effects
 				(font
@@
 				)
 				(justify left)
-			)
-		)
-		(property "Value" "TestPoint"
-			(at 83.82 85.5979 0)
-			(effects
-				(font
-					(size 1.27 1.27)
-				)
-				(justify left)
+				(hide yes)
 			)
 		)
 		(property "Footprint" "GoG_Library:TestPoint_Pad_D1.5mm_JLCPCB"
-			(at 86.36 87.63 0)
+			(at 93.98 76.2 0)
 			(effects
 				(font
@@
 		)
 		(property "Datasheet" "~"
-			(at 86.36 87.63 0)
+			(at 93.98 76.2 0)
 			(effects
 				(font
@@
 		)
 		(property "Description" "test point"
-			(at 81.28 87.63 0)
+			(at 93.98 81.28 0)
 			(effects
 				(font
@@
 			(project ""
 				(path "/5b969f6e-a36e-432b-8f00-b2d6a515a877/9db73a32-37a4-4249-8656-c1ba9b3afe01"
-					(reference "TP_RESET1")
+					(reference "TP1")
 					(unit 1)
 				)
@@
 	(symbol
 		(lib_id "power:GND")
-		(at 127 38.1 0)
+		(at 97.79 53.34 0)
 		(unit 1)
 		(exclude_from_sim no)
@@
 		(fields_autoplaced yes)
 		(property "Reference" "#PWR011"
-			(at 127 44.45 0)
+			(at 97.79 59.69 0)
 			(effects
 				(font
@@
 		)
 		(property "Value" "GND"
-			(at 127 43.18 0)
+			(at 97.79 58.42 0)
 			(effects
 				(font
@@
 		)
 		(property "Footprint" ""
-			(at 127 38.1 0)
+			(at 97.79 53.34 0)
 			(effects
 				(font
@@
 		)
 		(property "Datasheet" ""
-			(at 127 38.1 0)
+			(at 97.79 53.34 0)
 			(effects
 				(font
@@
 		)
 		(property "Description" "Power symbol creates a global label with name \"GND\" , ground"
-			(at 127 38.1 0)
+			(at 97.79 53.34 0)
 			(effects
 				(font
@@
 				(path "/5b969f6e-a36e-432b-8f00-b2d6a515a877/9db73a32-37a4-4249-8656-c1ba9b3afe01"
 					(reference "#PWR011")
-					(unit 1)
-				)
-			)
-		)
-	)
-	(symbol
-		(lib_id "Connector:TestPoint")
-		(at 92.71 50.8 0)
-		(unit 1)
-		(exclude_from_sim no)
-		(in_bom yes)
-		(on_board yes)
-		(dnp no)
-		(fields_autoplaced yes)
-		(property "Reference" "TP_VCC_Lora1"
-			(at 95.25 46.2279 0)
-			(effects
-				(font
-					(size 1.27 1.27)
-				)
-				(justify left)
-			)
-		)
-		(property "Value" "TestPoint"
-			(at 95.25 48.7679 0)
-			(effects
-				(font
-					(size 1.27 1.27)
-				)
-				(justify left)
-			)
-		)
-		(property "Footprint" "GoG_Library:TestPoint_Pad_D1.5mm_JLCPCB"
-			(at 97.79 50.8 0)
-			(effects
-				(font
-					(size 1.27 1.27)
-				)
-				(hide yes)
-			)
-		)
-		(property "Datasheet" "~"
-			(at 97.79 50.8 0)
-			(effects
-				(font
-					(size 1.27 1.27)
-				)
-				(hide yes)
-			)
-		)
-		(property "Description" "test point"
-			(at 92.71 50.8 0)
-			(effects
-				(font
-					(size 1.27 1.27)
-				)
-				(hide yes)
-			)
-		)
-		(pin "1"
-		)
-		(instances
-			(project ""
-				(path "/5b969f6e-a36e-432b-8f00-b2d6a515a877/9db73a32-37a4-4249-8656-c1ba9b3afe01"
-					(reference "TP_VCC_Lora1")
 					(unit 1)
 				)
@@
 	(symbol
 		(lib_id "Device:C")
-		(at 113.03 38.1 270)
+		(at 97.79 49.53 0)
 		(unit 1)
 		(exclude_from_sim no)
@@
 		(dnp no)
 		(property "Reference" "C4"
-			(at 114.3001 41.91 0)
+			(at 101.6 48.2599 0)
 			(effects
 				(font
@@
 		)
 		(property "Value" "100nF"
-			(at 111.7601 41.91 0)
+			(at 101.6 50.7999 0)
 			(effects
 				(font
@@
 		)
 		(property "Footprint" "Capacitor_SMD:C_0603_1608Metric"
-			(at 109.22 39.0652 0)
+			(at 98.7552 53.34 0)
 			(effects
 				(font
@@
 		)
 		(property "Datasheet" "~"
-			(at 113.03 38.1 0)
+			(at 97.79 49.53 0)
 			(effects
 				(font
@@
 		)
 		(property "Description" "100nF 25V X7R ±10% 0603 Multilayer Ceramic Capacitors MLCC - SMD/SMT ROHS"
-			(at 113.03 38.1 0)
+			(at 97.79 49.53 0)
 			(effects
 				(font
@@
 		)
 		(property "JLCPCB Part #" "C1590"
-			(at 113.03 38.1 0)
+			(at 97.79 49.53 0)
 			(effects
 				(font
@@
 		)
 		(property "Package" "0603"
-			(at 113.03 38.1 0)
-			(effects
-				(font
+			(at 97.79 49.53 0)
+			(effects
+				(font

Commit message: Find all remaining components on JLCPCB
Parts:
- C5, C6: value C -> (NC)
- R9: JLCPCB Part # / -> C2842889
- TP1, TP2: JLCPCB Part # (none) -> -; Package (none) -> -; now left out of the parts list
Changed lines of the file:
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@@
 		(unit 1)
 		(exclude_from_sim no)
-		(in_bom yes)
+		(in_bom no)
 		(on_board yes)
 		(dnp no)
@@
 			)
 		)
-		(property "Description" "test point"
+		(property "Description" "Test point 1.5mm diameter"
+			(at 125.73 81.28 0)
+			(effects
+				(font
+					(size 1.27 1.27)
+				)
+				(hide yes)
+			)
+		)
+		(property "JLCPCB Part #" "-"
+			(at 125.73 81.28 0)
+			(effects
+				(font
+					(size 1.27 1.27)
+				)
+				(hide yes)
+			)
+		)
+		(property "Package" "-"
 			(at 125.73 81.28 0)
 			(effects
@@
 			)
 		)
-		(property "Value" "C"
+		(property "Value" "(NC)"
 			(at 152.4 77.4699 0)
 			(effects
@@
 			)
 		)
-		(property "Description" "Resistor"
+		(property "Description" "PMR10EZPJ000 0Ω 500mW Shunt Resistor 0805"
 			(at 158.75 64.77 0)
 			(effects
@@
 			)
 		)
-		(property "JLCPCB Part #" "/"
+		(property "JLCPCB Part #" "C2842889"
 			(at 158.75 64.77 90)
 			(effects
@@
 		(unit 1)
 		(exclude_from_sim no)
-		(in_bom yes)
+		(in_bom no)
 		(on_board yes)
 		(dnp no)
@@
 			)
 		)
-		(property "Description" "test point"
+		(property "Description" "Test point 1.5mm diameter"
+			(at 93.98 81.28 0)
+			(effects
+				(font
+					(size 1.27 1.27)
+				)
+				(hide yes)
+			)
+		)
+		(property "JLCPCB Part #" "-"
+			(at 93.98 81.28 0)
+			(effects
+				(font
+					(size 1.27 1.27)
+				)
+				(hide yes)
+			)
+		)
+		(property "Package" "-"
 			(at 93.98 81.28 0)
 			(effects
@@
 			)
 		)
-		(property "Value" "C"
+		(property "Value" "(NC)"
 			(at 168.91 77.4699 0)
 			(effects
@@
 			)
 		)
-		(property "Description" "100nF 25V X7R ±10% 0603 Multilayer Ceramic Capacitors MLCC - SMD/SMT ROHS"
+		(property "Description" "CL10B104KA8NNNC 100nF 25V X7R ±10% 0603 Multilayer Ceramic Capacitors MLCC - SMD/SMT ROHS"
 			(at 97.79 49.53 0)
 			(effects
